Commit message: fix biped mesh labels

File: urdf/biped_with_mass.urdf (robot description, URDF)
Before this commit: robot biped, 7 links, 3 joints
Links:
- link L_hipassembly: geometry visual mesh filename=package://ETH_biped/meshes/leg/hipassembly.dae scale=1 1 1
- link L_lowerleg: geometry visual mesh filename=package://ETH_biped/meshes/leg/lowerleg.dae scale=1 1 1
- link L_upperleg: geometry visual mesh filename=package://ETH_biped/meshes/leg/upperleg.dae scale=1 1 1
- link R_hipassembly: geometry visual mesh filename=package://ETH_biped/meshes/leg/hipassembly.dae scale=1 1 1
- link R_lowerleg: geometry visual mesh filename=package://ETH_biped/meshes/leg/lowerleg.dae scale=1 1 1
- link R_upperleg: geometry visual mesh filename=package://ETH_biped/meshes/leg/upperleg.dae scale=1 1 1

Commit message: urdfs for blackbird, but I gotta debug

File: urdf/biped_with_mass.urdf (robot description, URDF)
Before this commit: robot biped, 7 links, 3 joints
Links:
- link L_hipassembly: geometry visual mesh filename=package://ETH_biped/meshes/ETH/leg/hipassembly.dae scale=1 1 1
- link L_lowerleg: geometry visual mesh filename=package://ETH_biped/meshes/ETH/leg/lowerleg.dae scale=1 1 1
- link L_upperleg: geometry visual mesh filename=package://ETH_biped/meshes/ETH/leg/upperleg.dae scale=1 1 1
- link R_hipassembly: geometry visual mesh filename=package://ETH_biped/meshes/ETH/leg/hipassembly.dae scale=1 1 1
- link R_lowerleg: geometry visual mesh filename=package://ETH_biped/meshes/ETH/leg/lowerleg.dae scale=1 1 1
- link R_upperleg: geometry visual mesh filename=package://ETH_biped/meshes/ETH/leg/upperleg.dae scale=1 1 1
