Commit message: test env for blackbird ready

File: urdf/blackbird_original.urdf (robot description, URDF)
Before this commit: robot blackbird, 12 links, 11 joints
Links:
- removed link world
- link l_ab_ad: geometry collision cylinder length=0.0759 radius=0.055; visual mesh filename=../meshes/stl/Assembly Mockup v27.003.stl scale=1.0 1.0 1.0
- link l_foot: geometry collision sphere radius=0.025; collision sphere radius=0.025
- link l_lower: geometry collision cylinder length=0.088 radius=0.055; visual mesh filename=../meshes/stl/Assembly Mockup v27.011.stl scale=1.0 1.0 1.0
- link l_upper: geometry visual mesh filename=../meshes/stl/Assembly Mockup v27.013.stl scale=1.0 1.0 1.0
- link l_yaw: geometry collision cylinder length=0.209 radius=0.0525; visual mesh filename=../meshes/stl/Assembly Mockup v27.005.stl scale=1.0 1.0 1.0
- link r_ab_ad: geometry collision cylinder length=0.0759 radius=0.055; visual mesh filename=../meshes/stl/Assembly Mockup v27.004.stl scale=1.0 1.0 1.0
- link r_foot: geometry collision sphere radius=0.025; collision sphere radius=0.025
- link r_lower: geometry collision cylinder length=0.088 radius=0.055; visual mesh filename=../meshes/stl/Assembly Mockup v27.010.stl scale=1.0 1.0 1.0
- link r_upper: geometry visual mesh filename=../meshes/stl/Assembly Mockup v27.009.stl scale=1.0 1.0 1.0
- link r_yaw: geometry collision cylinder length=0.209 radius=0.0525; visual mesh filename=../meshes/stl/Assembly Mockup v27.006.stl scale=1.0 1.0 1.0
- link torso: geometry collision box size=0.16028 0.33 0.145; collision cylinder length=0.0759 radius=0.055
Joints:
- removed joint l_ankle
- removed joint l_hip_pitch
- removed joint l_hip_roll
- removed joint l_hip_yaw
- removed joint l_knee
- removed joint r_ankle
- removed joint r_hip_pitch
- removed joint r_hip_roll
- removed joint r_hip_yaw
- removed joint r_knee
- removed joint world_to_torso
- added joint l_ab_ad: type revolute, parent torso, child l_ab_ad, origin xyz=0.15 0 0 rpy=0 0 0, axis 0 -1.0 0, limit lower=-2 upper=2 effort=0 velocity=0
- added joint l_foot: type revolute, parent l_lower, child l_foot, origin xyz=0 -0.1529 -0.42302 rpy=0 0 0, axis 1.0 0 0, limit lower=-1.5708 upper=0.69813 effort=0 velocity=0
- added joint l_lower: type revolute, parent l_upper, child l_lower, origin xyz=0 0.1529 -0.42302 rpy=0 0 0, axis 1.0 0 0, limit lower=-2.0944 upper=0.34907 effort=0 velocity=0
- added joint l_upper: type revolute, parent l_yaw, child l_upper, origin xyz=0 0 0 rpy=0 0 0, axis 1.0 0 0, limit lower=-1.91986 upper=1.22173 effort=0 velocity=0
- added joint l_yaw: type revolute, parent l_ab_ad, child l_yaw, origin xyz=0 0 -0.1295 rpy=0 0 0, axis 0 0 1.0, limit lower=-2 upper=2 effort=0 velocity=0
- added joint r_ab_ad: type revolute, parent torso, child r_ab_ad, origin xyz=-0.15 0 0 rpy=0 0 0, axis 0 -1.0 0, limit lower=-2 upper=2 effort=0 velocity=0
- added joint r_foot: type revolute, parent r_lower, child r_foot, origin xyz=0 -0.1529 -0.42302 rpy=0 0 0, axis 1.0 0 0, limit lower=-1.5708 upper=0.69813 effort=0 velocity=0
- added joint r_lower: type revolute, parent r_upper, child r_lower, origin xyz=0 0.1529 -0.42302 rpy=0 0 0, axis 1.0 0 0, limit lower=-2.0944 upper=0.34907 effort=0 velocity=0
- added joint r_upper: type revolute, parent r_yaw, child r_upper, origin xyz=0 0 0 rpy=0 0 0, axis 1.0 0 0, limit lower=-1.91986 upper=1.22173 effort=0 velocity=0
- added joint r_yaw: type revolute, parent r_ab_ad, child r_yaw, origin xyz=0 0 -0.1295 rpy=0 0 0, axis 0 0 1.0, limit lower=-2 upper=2 effort=0 velocity=0
