Commit message: fixed mesh file read bug by copying 'gym-ignition-models'

File: urdf/blackbird_ign.urdf (robot description, URDF)
Before this commit: robot blackbird, 12 links, 11 joints
Links:
- link l_ab_ad: geometry collision cylinder length=0.0759 radius=0.055; visual mesh filename=file://meshes/blackbird/Assembly_Mockup_v27_003.stl scale=1.0 1.0 1.0
- link l_foot: geometry collision sphere radius=0.025; collision sphere radius=0.025
- link l_lower: geometry collision cylinder length=0.088 radius=0.055; visual mesh filename=file://meshes/blackbird/Assembly_Mockup_v27_011.stl scale=1.0 1.0 1.0
- link l_upper: geometry visual mesh filename=file://meshes/blackbird/Assembly_Mockup_v27_013.stl scale=1.0 1.0 1.0
- link l_yaw: geometry collision cylinder length=0.209 radius=0.0525; visual mesh filename=file://meshes/blackbird/Assembly_Mockup_v27_005.stl scale=1.0 1.0 1.0
- link r_ab_ad: geometry collision cylinder length=0.0759 radius=0.055; visual mesh filename=file://meshes/blackbird/Assembly_Mockup_v27_004.stl scale=1.0 1.0 1.0
- link r_foot: geometry collision sphere radius=0.025; collision sphere radius=0.025
- link r_lower: geometry collision cylinder length=0.088 radius=0.055; visual mesh filename=file://meshes/blackbird/Assembly_Mockup_v27_010.stl scale=1.0 1.0 1.0
- link r_upper: geometry visual mesh filename=file://meshes/blackbird/Assembly_Mockup_v27_009.stl scale=1.0 1.0 1.0
- link r_yaw: geometry collision cylinder length=0.209 radius=0.0525; visual mesh filename=file://meshes/blackbird/Assembly_Mockup_v27_006.stl scale=1.0 1.0 1.0
- link torso: geometry collision box size=0.16028 0.33 0.145; collision cylinder length=0.0759 radius=0.055
Joints:
- joint world_to_torso: child slideBar -> torso; parent torso -> world

Commit message: spawn bipedal properly in ignition sim

File: urdf/blackbird_ign.urdf (robot description, URDF)
Before this commit: robot blackbird, 12 links, 11 joints
Links:
- removed link world
Joints:
- removed joint world_to_torso
