Commit message: blackbird rviz visualized

File: urdf/blackbird.urdf (robot description, URDF)
Before this commit: robot blackbird, 11 links, 10 joints
Links:
- link l_ab_ad: geometry collision cylinder length=0.0759 radius=0.055; visual mesh filename=package://ETH_biped/meshes/blackbird/Assembly_Mockup_v27_00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 scale=1.0 1.0 1.0
- link l_foot: geometry collision sphere radius=0.025; collision sphere radius=0.025
- link l_lower: geometry collision cylinder length=0.088 radius=0.055; visual mesh filename=package://ETH_biped/meshes/blackbird/Assembly_Mockup_v27_01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 scale=1.0 1.0 1.0
- link l_upper: geometry visual mesh filename=package://ETH_biped/meshes/blackbird/Assembly_Mockup_v27_01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 scale=1.0 1.0 1.0
- link l_yaw: geometry collision cylinder length=0.209 radius=0.0525; visual mesh filename=package://ETH_biped/meshes/blackbird/Assembly_Mockup_v27_00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 scale=1.0 1.0 1.0
- link r_ab_ad: geometry collision cylinder length=0.0759 radius=0.055; visual mesh filename=package://ETH_biped/meshes/blackbird/Assembly_Mockup_v27_00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 scale=1.0 1.0 1.0
- link r_foot: geometry collision sphere radius=0.025; collision sphere radius=0.025
- link r_lower: geometry collision cylinder length=0.088 radius=0.055; visual mesh filename=package://ETH_biped/meshes/blackbird/Assembly_Mockup_v27_01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 scale=1.0 1.0 1.0
- link r_upper: geometry visual mesh filename=package://ETH_biped/meshes/blackbird/Assembly_Mockup_v27_00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 scale=1.0 1.0 1.0
- link r_yaw: geometry collision cylinder length=0.209 radius=0.0525; visual mesh filename=package://ETH_biped/meshes/blackbird/Assembly_Mockup_v27_00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 scale=1.0 1.0 1.0
- link torso: geometry collision box size=0.16028 0.33 0.145; collision cylinder length=0.0759 radius=0.055

Commit message: attempted effort limits

File: urdf/blackbird.urdf (robot description, URDF)
Before this commit: robot blackbird, 11 links, 10 joints
Joints:
- joint l_ab_ad: limit lower=-2 upper=2 effort=0 velocity=0 -> lower=-2 upper=2 effort=50 velocity=20
- joint l_foot: limit lower=-1.5708 upper=0.69813 effort=0 velocity=0 -> lower=-1.5708 upper=0.69813 effort=50 velocity=20
- joint l_lower: limit lower=-2.0944 upper=0.34907 effort=0 velocity=0 -> lower=-2.0944 upper=0.34907 effort=50 velocity=20
- joint l_upper: limit lower=-1.91986 upper=1.22173 effort=0 velocity=0 -> lower=-1.91986 upper=1.22173 effort=50 velocity=20
- joint l_yaw: limit lower=-2 upper=2 effort=0 velocity=0 -> lower=-2 upper=2 effort=50 velocity=20
- joint r_ab_ad: limit lower=-2 upper=2 effort=0 velocity=0 -> lower=-2 upper=2 effort=50 velocity=20
- joint r_foot: limit lower=-1.5708 upper=0.69813 effort=0 velocity=0 -> lower=-1.5708 upper=0.69813 effort=50 velocity=20
- joint r_lower: limit lower=-2.0944 upper=0.34907 effort=0 velocity=0 -> lower=-2.0944 upper=0.34907 effort=50 velocity=20
- joint r_upper: limit lower=-1.91986 upper=1.22173 effort=0 velocity=0 -> lower=-1.91986 upper=1.22173 effort=50 velocity=20
- joint r_yaw: limit lower=-2 upper=2 effort=0 velocity=0 -> lower=-2 upper=2 effort=50 velocity=20

Commit message: added world 'dummy' link to enable better rviz and for gz fortress simulation

File: urdf/blackbird.urdf (robot description, URDF)
Before this commit: robot blackbird, 11 links, 10 joints
Links:
- added link world
Joints:
- added joint world_to_torso: type fixed, parent world, child torso, origin xyz=0 0 1 rpy=0 0 0

File: urdf/blackbird_ign.urdf (robot description, URDF)
Before this commit: robot blackbird, 11 links, 10 joints
Links:
- added link world
Joints:
- added joint world_to_torso: type fixed, parent torso, child slideBar, origin xyz=0 0 1 rpy=0 0 0

Commit message: ingition launch

File: urdf/blackbird.urdf (robot description, URDF)
Before this commit: robot blackbird, 12 links, 11 joints
Joints:
- removed joint l_ab_ad
- removed joint l_foot
- removed joint l_lower
- removed joint l_upper
- removed joint l_yaw
- removed joint r_ab_ad
- removed joint r_foot
- removed joint r_lower
- removed joint r_upper
- removed joint r_yaw
- added joint l_ankle: type revolute, parent l_lower, child l_foot, origin xyz=0 -0.1529 -0.42302 rpy=0 0 0, axis 1.0 0 0, limit lower=-1.5708 upper=0.69813 effort=50 velocity=20
- added joint l_hip_pitch: type revolute, parent torso, child l_ab_ad, origin xyz=0.15 0 0 rpy=0 0 0, axis 0 -1.0 0, limit lower=-2 upper=2 effort=50 velocity=20
- added joint l_hip_roll: type revolute, parent l_yaw, child l_upper, origin xyz=0 0 0 rpy=0 0 0, axis 1.0 0 0, limit lower=-1.91986 upper=1.22173 effort=50 velocity=20
- added joint l_hip_yaw: type revolute, parent l_ab_ad, child l_yaw, origin xyz=0 0 -0.1295 rpy=0 0 0, axis 0 0 1.0, limit lower=-2 upper=2 effort=50 velocity=20
- added joint l_knee: type revolute, parent l_upper, child l_lower, origin xyz=0 0.1529 -0.42302 rpy=0 0 0, axis 1.0 0 0, limit lower=-2.0944 upper=0.34907 effort=50 velocity=20
- added joint r_ankle: type revolute, parent r_lower, child r_foot, origin xyz=0 -0.1529 -0.42302 rpy=0 0 0, axis 1.0 0 0, limit lower=-1.5708 upper=0.69813 effort=50 velocity=20
- added joint r_hip_pitch: type revolute, parent torso, child r_ab_ad, origin xyz=-0.15 0 0 rpy=0 0 0, axis 0 -1.0 0, limit lower=-2 upper=2 effort=50 velocity=20
- added joint r_hip_roll: type revolute, parent r_yaw, child r_upper, origin xyz=0 0 0 rpy=0 0 0, axis 1.0 0 0, limit lower=-1.91986 upper=1.22173 effort=50 velocity=20
- added joint r_hip_yaw: type revolute, parent r_ab_ad, child r_yaw, origin xyz=0 0 -0.1295 rpy=0 0 0, axis 0 0 1.0, limit lower=-2 upper=2 effort=50 velocity=20
- added joint r_knee: type revolute, parent r_upper, child r_lower, origin xyz=0 0.1529 -0.42302 rpy=0 0 0, axis 1.0 0 0, limit lower=-2.0944 upper=0.34907 effort=50 velocity=20

Commit message: effort controllers working and are functional

File: urdf/blackbird.urdf (robot description, URDF)
Before this commit: robot blackbird, 12 links, 11 joints
Joints:
- joint l_hip_pitch: axis 0 -1.0 0 -> 1.0 0 0; child l_ab_ad -> l_upper; limit lower=-2 upper=2 effort=50 velocity=20 -> lower=-1.91986 upper=1.22173 effort=50 velocity=20; origin xyz=0.15 0 0 rpy=0 0 0 -> xyz=0 0 0 rpy=0 0 0; parent torso -> l_yaw
- joint l_hip_roll: axis 1.0 0 0 -> 0 -1.0 0; child l_upper -> l_ab_ad; limit lower=-1.91986 upper=1.22173 effort=50 velocity=20 -> lower=-2 upper=2 effort=50 velocity=20; origin xyz=0 0 0 rpy=0 0 0 -> xyz=0.15 0 0 rpy=0 0 0; parent l_yaw -> torso
- joint r_hip_pitch: axis 0 -1.0 0 -> 1.0 0 0; child r_ab_ad -> r_upper; limit lower=-2 upper=2 effort=50 velocity=20 -> lower=-1.91986 upper=1.22173 effort=50 velocity=20; origin xyz=-0.15 0 0 rpy=0 0 0 -> xyz=0 0 0 rpy=0 0 0; parent torso -> r_yaw
- joint r_hip_roll: axis 1.0 0 0 -> 0 -1.0 0; child r_upper -> r_ab_ad; limit lower=-1.91986 upper=1.22173 effort=50 velocity=20 -> lower=-2 upper=2 effort=50 velocity=20; origin xyz=0 0 0 rpy=0 0 0 -> xyz=-0.15 0 0 rpy=0 0 0; parent r_yaw -> torso

File: urdf/blackbird_ign.urdf (robot description, URDF)
Before this commit: robot blackbird, 12 links, 11 joints
Joints:
- joint l_hip_pitch: axis 0 -1.0 0 -> 1.0 0 0; child l_ab_ad -> l_upper; limit lower=-2 upper=2 effort=50 velocity=20 -> lower=-1.91986 upper=1.22173 effort=50 velocity=20; origin xyz=0.15 0 0 rpy=0 0 0 -> xyz=0 0 0 rpy=0 0 0; parent torso -> l_yaw
- joint l_hip_roll: axis 1.0 0 0 -> 0 -1.0 0; child l_upper -> l_ab_ad; limit lower=-1.91986 upper=1.22173 effort=50 velocity=20 -> lower=-2 upper=2 effort=50 velocity=20; origin xyz=0 0 0 rpy=0 0 0 -> xyz=0.15 0 0 rpy=0 0 0; parent l_yaw -> torso
- joint r_hip_pitch: axis 0 -1.0 0 -> 1.0 0 0; child r_ab_ad -> r_upper; limit lower=-2 upper=2 effort=50 velocity=20 -> lower=-1.91986 upper=1.22173 effort=50 velocity=20; origin xyz=-0.15 0 0 rpy=0 0 0 -> xyz=0 0 0 rpy=0 0 0; parent torso -> r_yaw
- joint r_hip_roll: axis 1.0 0 0 -> 0 -1.0 0; child r_upper -> r_ab_ad; limit lower=-1.91986 upper=1.22173 effort=50 velocity=20 -> lower=-2 upper=2 effort=50 velocity=20; origin xyz=0 0 0 rpy=0 0 0 -> xyz=-0.15 0 0 rpy=0 0 0; parent r_yaw -> torso

Commit message: making this repo blackbird only...just have to confirm blackbird_ign launches properly

File: urdf/blackbird.urdf (robot description, URDF)
Before this commit: robot blackbird, 12 links, 11 joints
Links:
- link l_ab_ad: geometry collision cylinder length=0.0759 radius=0.055; visual mesh filename=package://blackbird_ros2/meshes/blackbird/Assembly_Mockup_v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 scale=1.0 1.0 1.0
- link l_foot: geometry collision sphere radius=0.025; collision sphere radius=0.025
- link l_lower: geometry collision cylinder length=0.088 radius=0.055; visual mesh filename=package://blackbird_ros2/meshes/blackbird/Assembly_Mockup_v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 scale=1.0 1.0 1.0
- link l_upper: geometry visual mesh filename=package://blackbird_ros2/meshes/blackbird/Assembly_Mockup_v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 scale=1.0 1.0 1.0
- link l_yaw: geometry collision cylinder length=0.209 radius=0.0525; visual mesh filename=package://blackbird_ros2/meshes/blackbird/Assembly_Mockup_v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 scale=1.0 1.0 1.0
- link r_ab_ad: geometry collision cylinder length=0.0759 radius=0.055; visual mesh filename=package://blackbird_ros2/meshes/blackbird/Assembly_Mockup_v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 scale=1.0 1.0 1.0
- link r_foot: geometry collision sphere radius=0.025; collision sphere radius=0.025
- link r_lower: geometry collision cylinder length=0.088 radius=0.055; visual mesh filename=package://blackbird_ros2/meshes/blackbird/Assembly_Mockup_v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 scale=1.0 1.0 1.0
- link r_upper: geometry visual mesh filename=package://blackbird_ros2/meshes/blackbird/Assembly_Mockup_v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 scale=1.0 1.0 1.0
- link r_yaw: geometry collision cylinder length=0.209 radius=0.0525; visual mesh filename=package://blackbird_ros2/meshes/blackbird/Assembly_Mockup_v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 scale=1.0 1.0 1.0
- link torso: geometry collision box size=0.16028 0.33 0.145; collision cylinder length=0.0759 radius=0.055
