Commit message: fixed up joint order in urdf for explanations

File: urdf/blackbird_gz.urdf (robot description, URDF)
Before this commit: robot blackbird, 11 links, 10 joints
Joints:
- joint l_hip_pitch: axis 1.0 0 0 -> 0 0 1.0; child l_upper -> l_yaw; limit lower=-1.91986 upper=1.22173 effort=50 velocity=20 -> lower=-2 upper=2 effort=50 velocity=20; origin xyz=0 0 0 rpy=0 0 0 -> xyz=0 0 -0.1295 rpy=0 0 0; parent l_yaw -> l_ab_ad
- joint l_hip_yaw: axis 0 0 1.0 -> 1.0 0 0; child l_yaw -> l_upper; limit lower=-2 upper=2 effort=50 velocity=20 -> lower=-1.91986 upper=1.22173 effort=50 velocity=20; origin xyz=0 0 -0.1295 rpy=0 0 0 -> xyz=0 0 0 rpy=0 0 0; parent l_ab_ad -> l_yaw
- joint r_hip_pitch: axis 1.0 0 0 -> 0 0 1.0; child r_upper -> r_yaw; limit lower=-1.91986 upper=1.22173 effort=50 velocity=20 -> lower=-2 upper=2 effort=50 velocity=20; origin xyz=0 0 0 rpy=0 0 0 -> xyz=0 0 -0.1295 rpy=0 0 0; parent r_yaw -> r_ab_ad
- joint r_hip_yaw: axis 0 0 1.0 -> 1.0 0 0; child r_yaw -> r_upper; limit lower=-2 upper=2 effort=50 velocity=20 -> lower=-1.91986 upper=1.22173 effort=50 velocity=20; origin xyz=0 0 -0.1295 rpy=0 0 0 -> xyz=0 0 0 rpy=0 0 0; parent r_ab_ad -> r_yaw
